File: schematics/PCBs/2-to-4 Selector/Transistor 2-to-4 Selector.kicad_sch (KiCad schematic)
At the start: 62 parts, among them J1 EN, J10 EN4, J2 D0, J3 Power, J4 Power, J5 Power, J6 D1, J7 EN1, J8 EN2, J9 EN3, Q1 2N2222, Q10 2N2222, Q11 2N2222, Q12 2N2222, Q13 2N2222, Q14 2N2222, Q15 2N2222, Q16 2N2222, Q17 2N2222, Q18 2N2222, Q19 2N2222, Q2 2N2222, Q20 2N2222, Q21 2N2222, Q22 2N2222, Q23 2N2222, Q3 2N2222, Q4 2N2222, Q5 2N2222, Q6 2N2222, Q7 2N2222, Q8 2N2222, Q9 2N2222

Commit message: Update schematic based on in-the-field rework necessary with new transistor supplier.
Parts:
- R10, R11, R12, R9: value 1K -> 10K
Changed lines of the file:
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@@
       (effects (font (size 1.27 1.27)) (justify left))
     )
-    (property "Value" "1K" (at 131.318 62.103 0)
+    (property "Value" "10K" (at 131.318 62.103 0)
       (effects (font (size 1.27 1.27)) (justify left))
     )
@@
       (effects (font (size 1.27 1.27)) (justify left))
     )
-    (property "Value" "1K" (at 131.318 92.583 0)
+    (property "Value" "10K" (at 131.318 92.583 0)
       (effects (font (size 1.27 1.27)) (justify left))
     )
@@
       (effects (font (size 1.27 1.27)) (justify left))
     )
-    (property "Value" "1K" (at 131.318 126.873 0)
+    (property "Value" "10K" (at 131.318 126.873 0)
       (effects (font (size 1.27 1.27)) (justify left))
     )
@@
       (effects (font (size 1.27 1.27)) (justify left))
     )
-    (property "Value" "1K" (at 131.318 157.353 0)
-      (effects (font (size 1.27 1.27)) (justify left))
-    )
+    (property "Value" "10K" (at 131.318 157.353 0)
+      (effects (font (size 1.27 1.27)) (justify left))
+    )
