File: schematics/Layout/ALU.kicad_sch (KiCad schematic)
At the start: 11 parts

Commit message: Update README with progress, update layout with new instruction decoder board.
Connections:
- new net: B55. (EN2), B57. (EN4)
- new net: B55. (EN2), B56. (EN4)
- new net: B59. (NONZERO), B60. (OUT)
