File: schematics/Layout/D Register.kicad_sch (KiCad schematic)
At the start: 7 parts

Commit message: Update README with progress, update layout with new instruction decoder board.
Connections:
- new net: B11. (OUT4), B13. (OUT8), B14. (OUT8) (x4)
- new net: B11. (OUT4), B12. (OUT4), B146. (OUT)
- new net: B12. (OUT4), B13. (OUT8), B14. (OUT8) (x4)
- new net: B13. (OUT8), B148. (OUT)
- new net: B14. (OUT8), B147. (OUT)
Changed lines of the file:
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@@
 	)
 	(symbol
-		(lib_name "4-Bit Register_1")
 		(lib_id "MiniDragon:4-Bit Register")
 		(at 99.06 149.86 0)
@@
 	)
 	(symbol
+		(lib_name "8-bit Bus Output_1")
 		(lib_id "MiniDragon:8-bit Bus Output")
 		(at 168.91 86.36 0)
@@
 	)
 	(symbol
-		(lib_name "Logic Buffer_2")
+		(lib_name "Logic Buffer_1")
 		(lib_id "MiniDragon:Logic Buffer")
 		(at 100.33 57.15 0)
@@
 	)
 	(symbol
-		(lib_name "8-bit Bus Output_1")
 		(lib_id "MiniDragon:8-bit Bus Output")
 		(at 168.91 137.16 0)
@@
 	)
 	(symbol
-		(lib_name "Logic Buffer_1")
+		(lib_name "Logic Buffer_2")
 		(lib_id "MiniDragon:Logic Buffer")
 		(at 100.33 35.56 0)
@@
 	)
 	(symbol
+		(lib_name "4-Bit Register_1")
 		(lib_id "MiniDragon:4-Bit Register")
 		(at 100.33 88.9 0)
