File: schematics/Layout/Immediate Register.kicad_sch (KiCad schematic)
At the start: 6 parts

Commit message: Update README with progress, update layout with new instruction decoder board.
Connections:
- new net: B129. (OUT), B27. (OUT8)
- new net: B127. (OUT), B25. (OUT8)
- new net: B128. (OUT), B26. (OUT8)
