File: schematics/Layout/SRAM Interface.kicad_sch (KiCad schematic)
At the start: 5 parts

Commit message: Update README with progress, update layout with new instruction decoder board.
Connections:
- new net: B156. (OUT8), B157. (OUT8) (x8)
Changed lines of the file:
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@@
 	)
 	(symbol
+		(lib_name "8-bit Logic Buffer_1")
 		(lib_id "MiniDragon:8-bit Logic Buffer")
 		(at 53.34 82.55 0)
@@
 	)
 	(symbol
-		(lib_name "8-bit Logic Buffer_1")
 		(lib_id "MiniDragon:8-bit Logic Buffer")
 		(at 53.34 34.29 0)
